File: mtf122.kicad_pcb (KiCad board)
At the start: 2 copper layers, 500 x 194 mm, 192 parts, among them J1 CONN_CAP_IBM_F, SW1 1,8, SW10 A,8, SW100 6,2, SW101 7,2, SW102 7,1, SW103 8,2, SW104 9,1, SW105 A,1, SW106 A,2, SW107 B,2, SW108 C,2, SW109 D,2, SW11 B,8, SW110 D,3, SW111 E,3, SW112 E,2, SW113 F,3, SW114 G,3, SW115 G,2, SW116 1,1, SW117 2,1, SW118 3,1, SW119 4,1, SW12 C,8, SW120 6,1, SW121 8,1, SW122 C,1, SW123 D,1, SW124 E,1, SW125 F,1, SW126 F,2, SW127 G,1, SW13 1,7, SW14 2,7, SW15 3,7, SW16 4,7, SW17 5,7, SW18 6,7, SW19 7,7, SW2 2,8, SW20 8,7, SW21 9,7, SW22 A,7, SW23 B,7, SW24 C,7, SW25 1,5, SW26 1,6, SW27 2,6, SW28 3,6, SW29 4,6, SW3 3,8, SW30 5,6, SW31 5,5, SW32 6,6, SW33 7,6, SW34 8,5, SW35 8,6, SW36 9,6, SW37 9,5, SW38 A,6, SW39 B,6, SW4 4,8, SW40 C,6, SW41 D,7, SW42 D,8, SW43 E,7, SW44 E,8, SW45 F,7, SW46 F,8, SW47 G,7, SW48 G,8, SW49 1,4, SW5 5,8, SW50 2,4, SW51 2,5, SW52 3,5, SW53 4,5, SW54 5,4, SW55 6,5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

Commit message: Removed redundant edge
Changed lines of the file:
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@@
   (general
     (thickness 0.8)
-    (drawings 60)
+    (drawings 58)
     (tracks 2562)
     (zones 0)
@@
     (0 F.Cu signal hide)
     (31 B.Cu signal hide)
-    (32 B.Adhes user)
-    (33 F.Adhes user)
-    (34 B.Paste user)
-    (35 F.Paste user)
-    (36 B.SilkS user)
-    (37 F.SilkS user)
+    (32 B.Adhes user hide)
+    (33 F.Adhes user hide)
+    (34 B.Paste user hide)
+    (35 F.Paste user hide)
+    (36 B.SilkS user hide)
+    (37 F.SilkS user hide)
     (38 B.Mask user)
     (39 F.Mask user)
-    (40 Dwgs.User user)
-    (41 Cmts.User user)
-    (42 Eco1.User user)
-    (43 Eco2.User user)
+    (40 Dwgs.User user hide)
+    (41 Cmts.User user hide)
+    (42 Eco1.User user hide)
+    (43 Eco2.User user hide)
     (44 Edge.Cuts user)
-    (45 Margin user)
-    (46 B.CrtYd user)
-    (47 F.CrtYd user)
-    (48 B.Fab user)
-    (49 F.Fab user)
+    (45 Margin user hide)
+    (46 B.CrtYd user hide)
+    (47 F.CrtYd user hide)
+    (48 B.Fab user hide)
+    (49 F.Fab user hide)
   )
   (setup
@@
     (visible_elements 7FFFFFFF)
     (pcbplotparams
-      (layerselection 0x210f0_ffffffff)
+      (layerselection 0x010c0_7ffffffe)
       (usegerberextensions false)
       (usegerberattributes true)
@@
       (creategerberjobfile true)
       (excludeedgelayer false)
-      (linewidth 0.150000)
+      (linewidth 1.000000)
       (plotframeref false)
       (viasonmask false)
       (mode 1)
-      (useauxorigin true)
+      (useauxorigin false)
       (hpglpennumber 1)
       (hpglpenspeed 20)
@@
       (psnegative false)
       (psa4output false)
-      (plotreference true)
-      (plotvalue true)
+      (plotreference false)
+      (plotvalue false)
       (plotinvisibletext false)
       (padsonsilk true)
       (subtractmaskfromsilk false)
-      (outputformat 1)
+      (outputformat 4)
       (mirror false)
-      (drillshape 0)
+      (drillshape 2)
       (scaleselection 1)
       (outputdirectory "gerber/"))
@@
   )
   (gr_line (start 47.523056 299.009113) (end 50.523056 302.009113) (layer Edge.Cuts) (width 0.1))
-  (gr_line (start 547.523056 299.009113) (end 547.523056 162.509113) (layer Edge.Cuts) (width 0.1))
   (gr_line (start 544.523056 302.009113) (end 547.523056 299.009113) (layer Edge.Cuts) (width 0.1))
   (gr_line (start 544.523056 159.509113) (end 547.523056 162.509113) (layer Edge.Cuts) (width 0.1))
-  (gr_line (start 47.523056 182.509113) (end 47.523056 299.009113) (layer Edge.Cuts) (width 0.1))
   (gr_line (start 396.023056 166.509113) (end 396.023056 111.013635) (layer Edge.Cuts) (width 0.1))
   (gr_line (start 544.523056 159.509113) (end 409.023056 159.509113) (layer Edge.Cuts) (width 0.1))

Commit message: Updated traces and copper fill areas
Routing:
- net GND: track 9430.5 -> 9355.8 mm
- net COL_G: track 183.9 -> 175.2 mm
- net COL_F: track 177.7 -> 181.6 mm
- net COL_E: track 239.1 -> 242.9 mm
- net ROW_8: track 1085.0 -> 1087.6 mm
- net ROW_7: track 1059.4 -> 1062.0 mm

Commit message: Added extra connection to be compliant with IBM rule: all rows and columns must cross exactly the same number of times
Routing:
- net GND: track 9355.8 -> 9402.9 mm
- net ROW_1: track 1258.9 -> 1291.3 mm
- net ROW_7: track 1062.0 -> 1090.6 mm
- net ROW_3: track 1229.8 -> 1258.3 mm
- net ROW_6: track 1127.6 -> 1156.1 mm
- net COL_9: track 440.2 -> 455.6 mm
- net COL_5: track 504.8 -> 518.8 mm
- net COL_7: track 475.7 -> 487.8 mm
- net COL_A: track 424.4 -> 435.6 mm
- net ROW_4: track 1238.5 -> 1248.0 mm
- net ROW_5: track 1172.9 -> 1173.6 mm
- net ROW_2: track 1276.1 -> 1276.8 mm
- net ROW_8: track 1087.6 -> 1088.4 mm

Commit message: Made the PCB corners rounded
Changed lines of the file:
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@@
   (page A2)
   (layers
-    (0 F.Cu signal hide)
-    (31 B.Cu signal hide)
+    (0 F.Cu signal)
+    (31 B.Cu signal)
     (32 B.Adhes user hide)
     (33 F.Adhes user hide)
@@
       (effects (font (size 1 1) (thickness 0.15)))
     )
-    (fp_line (start 1.8 -1.8) (end -1.8 -1.8) (layer F.CrtYd) (width 0.05))
-    (fp_line (start 1.8 116.64) (end 1.8 -1.8) (layer F.CrtYd) (width 0.05))
-    (fp_line (start -1.8 116.64) (end 1.8 116.64) (layer F.CrtYd) (width 0.05))
-    (fp_line (start -1.8 -1.8) (end -1.8 116.64) (layer F.CrtYd) (width 0.05))
-    (fp_line (start -1.33 -1.33) (end 0 -1.33) (layer F.SilkS) (width 0.12))
-    (fp_line (start -1.33 0) (end -1.33 -1.33) (layer F.SilkS) (width 0.12))
-    (fp_line (start -1.33 1.27) (end 1.33 1.27) (layer F.SilkS) (width 0.12))
-    (fp_line (start 1.33 1.27) (end 1.33 116.17) (layer F.SilkS) (width 0.12))
-    (fp_line (start -1.33 1.27) (end -1.33 116.17) (layer F.SilkS) (width 0.12))
-    (fp_line (start -1.33 116.17) (end 1.33 116.17) (layer F.SilkS) (width 0.12))
-    (fp_line (start -1.27 -0.635) (end -0.635 -1.27) (layer F.Fab) (width 0.1))
-    (fp_line (start -1.27 116.11) (end -1.27 -0.635) (layer F.Fab) (width 0.1))
-    (fp_line (start 1.27 116.11) (end -1.27 116.11) (layer F.Fab) (width 0.1))
-    (fp_line (start 1.27 -1.27) (end 1.27 116.11) (layer F.Fab) (width 0.1))
     (fp_line (start -0.635 -1.27) (end 1.27 -1.27) (layer F.Fab) (width 0.1))
+    (fp_line (start 1.27 -1.27) (end 1.27 116.11) (layer F.Fab) (width 0.1))
+    (fp_line (start 1.27 116.11) (end -1.27 116.11) (layer F.Fab) (width 0.1))
+    (fp_line (start -1.27 116.11) (end -1.27 -0.635) (layer F.Fab) (width 0.1))
+    (fp_line (start -1.27 -0.635) (end -0.635 -1.27) (layer F.Fab) (width 0.1))
+    (fp_line (start -1.33 116.17) (end 1.33 116.17) (layer F.SilkS) (width 0.12))
+    (fp_line (start -1.33 1.27) (end -1.33 116.17) (layer F.SilkS) (width 0.12))
+    (fp_line (start 1.33 1.27) (end 1.33 116.17) (layer F.SilkS) (width 0.12))
+    (fp_line (start -1.33 1.27) (end 1.33 1.27) (layer F.SilkS) (width 0.12))
+    (fp_line (start -1.33 0) (end -1.33 -1.33) (layer F.SilkS) (width 0.12))
+    (fp_line (start -1.33 -1.33) (end 0 -1.33) (layer F.SilkS) (width 0.12))
+    (fp_line (start -1.8 -1.8) (end -1.8 116.64) (layer F.CrtYd) (width 0.05))
+    (fp_line (start -1.8 116.64) (end 1.8 116.64) (layer F.CrtYd) (width 0.05))
+    (fp_line (start 1.8 116.64) (end 1.8 -1.8) (layer F.CrtYd) (width 0.05))
+    (fp_line (start 1.8 -1.8) (end -1.8 -1.8) (layer F.CrtYd) (width 0.05))
     (fp_text user %R (at 0 36.83) (layer F.Fab)
       (effects (font (size 1 1) (thickness 0.15)))
@@
     (pad "" np_thru_hole circle (at 1.3575 0) (size 3.5 3.5) (drill 3.5) (layers *.Cu *.Mask))
   )
-  (gr_line (start 403.023056 169.509113) (end 406.023056 166.509113) (layer Edge.Cuts) (width 0.1))
-  (gr_line (start 396.023056 166.509113) (end 399.023056 169.509113) (layer Edge.Cuts) (width 0.1))
-  (gr_line (start 406.023056 162.509113) (end 409.023056 159.509113) (layer Edge.Cuts) (width 0.1))
-  (gr_line (start 393.023056 108.013635) (end 396.023056 111.013635) (layer Edge.Cuts) (width 0.1))
-  (gr_line (start 95.023056 111.013635) (end 98.023056 108.013635) (layer Edge.Cuts) (width 0.1))
-  (gr_line (start 92.023056 179.509113) (end 95.023056 176.509113) (layer Edge.Cuts) (width 0.1))
-  (gr_line (start 47.523056 182.509113) (end 50.523056 179.509113) (layer Edge.Cuts) (width 0.1))
-  (gr_line (start 47.523056 299.009113) (end 50.523056 302.009113) (layer Edge.Cuts) (width 0.1))
-  (gr_line (start 544.523056 302.009113) (end 547.523056 299.009113) (layer Edge.Cuts) (width 0.1))
-  (gr_line (start 544.523056 159.509113) (end 547.523056 162.509113) (layer Edge.Cuts) (width 0.1))
+  (gr_line (start 406.095487 166.380856) (end 406.095487 162.380856) (layer Edge.Cuts) (width 0.1))
+  (gr_line (start 399.095487 169.380856) (end 403.095487 169.380856) (layer Edge.Cuts) (width 0.1))
+  (gr_line (start 544.595487 159.380856) (end 409.095487 159.380856) (layer Edge.Cuts) (width 0.1))
+  (gr_line (start 396.095487 166.380856) (end 396.095487 110.885378) (layer Edge.Cuts) (width 0.1))
+  (gr_arc (start 393.095487 110.885378) (end 396.095487 110.885378) (angle -90) (layer Edge.Cuts) (width 0.1))
+  (gr_arc (start 98.095487 110.885378) (end 98.095487 107.885378) (angle -90) (layer Edge.Cuts) (width 0.1))
+  (gr_arc (start 50.595487 298.880856) (end 47.595487 298.880856) (angle -90) (layer Edge.Cuts) (width 0.1))
+  (gr_arc (start 544.595487 298.880856) (end 544.595487 301.880856) (angle -90) (layer Edge.Cuts) (width 0.1))
+  (gr_arc (start 544.595487 162.380856) (end 547.595487 162.380856) (angle -90) (layer Edge.Cuts) (width 0.1))
+  (gr_arc (start 409.095487 162.380856) (end 409.095487 159.380856) (angle -90) (layer Edge.Cuts) (width 0.1))
+  (gr_arc (start 403.095487 166.380856) (end 403.095487 169.380856) (angle -90) (layer Edge.Cuts) (width 0.1))
+  (gr_arc (start 399.095487 166.380856) (end 396.095487 166.380856) (angle -90) (layer Edge.Cuts) (width 0.1))
+  (gr_line (start 393.095487 107.885378) (end 98.095487 107.885378) (layer Edge.Cuts) (width 0.1))
+  (gr_line (start 409.095487 159.380856) (end 409.095487 159.380856) (layer Edge.Cuts) (width 0.1))
+  (gr_line (start 95.095487 176.380856) (end 95.095487 110.885378) (layer Edge.Cuts) (width 0.1))
+  (gr_line (start 50.595487 179.380856) (end 92.095487 179.380856) (layer Edge.Cuts) (width 0.1))
+  (gr_line (start 47.595487 298.880856) (end 47.595487 182.380856) (layer Edge.Cuts) (width 0.1))
+  (gr_arc (start 92.095487 176.380856) (end 92.095487 179.380856) (angle -90) (layer Edge.Cuts) (width 0.1))
+  (gr_arc (start 50.595487 182.380856) (end 50.595487 179.380856) (angle -90) (layer Edge.Cuts) (width 0.1))
+  (gr_line (start 50.595487 301.880856) (end 544.595487 301.880856) (layer Edge.Cuts) (width 0.1))
+  (gr_line (start 547.595487 298.880856) (end 547.595487 162.380856) (layer Edge.Cuts) (width 0.1))
   (gr_text CE (at 518.65 167.06 90) (layer F.SilkS)
     (effects (font (size 1 1) (thickness 0.15)) (justify left))
@@
     (effects (font (size 1 1) (thickness 0.15)) (justify left))
   )
-  (gr_line (start 396.023056 166.509113) (end 396.023056 111.013635) (layer Edge.Cuts) (width 0.1))
-  (gr_line (start 544.523056 159.509113) (end 409.023056 159.509113) (layer Edge.Cuts) (width 0.1))
-  (gr_line (start 547.523056 299.009113) (end 547.523056 162.509113) (layer Edge.Cuts) (width 0.1))
-  (gr_line (start 95.023056 176.509113) (end 95.023056 111.013635) (layer Edge.Cuts) (width 0.1))
-  (gr_line (start 50.523056 179.509113) (end 92.023056 179.509113) (layer Edge.Cuts) (width 0.1))
-  (gr_line (start 393.023056 108.013635) (end 98.023056 108.013635) (layer Edge.Cuts) (width 0.1))
-  (gr_line (start 409.023056 159.509113) (end 409.023056 159.509113) (layer Edge.Cuts) (width 0.1))
-  (gr_line (start 406.023056 166.509113) (end 406.023056 162.509113) (layer Edge.Cuts) (width 0.1))
-  (gr_line (start 399.023056 169.509113) (end 403.023056 169.509113) (layer Edge.Cuts) (width 0.1))
-  (gr_line (start 50.523056 302.009113) (end 544.523056 302.009113) (layer Edge.Cuts) (width 0.1))
-  (gr_line (start 47.523056 299.009113) (end 47.523056 182.509113) (layer Edge.Cuts) (width 0.1))
   (gr_text "For Manufacturer:\nIt is okay if the board will warp.  The board will be curved to shape by the customer and any warping will be corrected." (at 110 90) (layer F.Fab)
     (effects (font (size 2.54 2.54) (thickness 0.3)) (justify left))
@@
       (pts
         (xy 103.070591 114.804511) (xy 387.88 114.79) (xy 388.955148 115.829878) (xy 388.87 170.64) (xy 394.717433 176.421678)
-        (xy 407.35 176.41) (xy 413.34 170.25) (xy 450.103602 170.243247) (xy 460.596398 159.456753) (xy 544.580591 159.504511)
-        (xy 547.580591 162.504511) (xy 547.575591 189.834511) (xy 504.98 189.67) (xy 502.76 187.52) (xy 498.84 187.51)
+        (xy 407.35 176.41) (xy 413.34 170.25) (xy 450.103602 170.243247) (xy 460.77 158.79) (xy 548.16 158.79)
+        (xy 548.19 162.47) (xy 548.36 189.8) (xy 504.98 189.67) (xy 502.76 187.52) (xy 498.84 187.51)
         (xy 496.5 189.67) (xy 458 189.68) (xy 455.77 187.5) (xy 451.84 187.49) (xy 449.51 189.6)
         (xy 420.02 189.68) (xy 417.74 187.46) (xy 413.85 187.463519) (xy 411.5 189.68) (xy 383.3 189.66)
@@
     (polygon
       (pts
-        (xy 396.074751 111.109689) (xy 396.154751 166.579689) (xy 399.154751 169.579689) (xy 403.114751 169.469689) (xy 406.084751 166.539689)
-        (xy 406.084751 162.539689) (xy 409.094751 159.539689) (xy 468.4 159.48) (xy 454.23 173.71) (xy 414.12 173.73)
+        (xy 396.82 111.05) (xy 396.81 166.51) (xy 399.03 168.75) (xy 403 168.81) (xy 405.38 166.31)
+        (xy 405.38 158.71) (xy 409.07 158.8) (xy 468.61 158.93) (xy 454.23 173.71) (xy 414.12 173.73)
         (xy 407.69 180.16) (xy 391.254751 180.209689) (xy 377.204751 166.119689) (xy 377.224751 138.679689) (xy 357.764751 119.269689)
         (xy 126.214751 119.089689) (xy 126.254751 131.549689) (xy 126.074751 186.989689) (xy 106.754751 187.029689) (xy 92.964751 200.999689)
-        (xy 60.184751 200.939689) (xy 60.284751 302.049689) (xy 50.564751 302.049689) (xy 47.584751 299.039689) (xy 47.584751 182.569689)
-        (xy 50.594751 179.559689) (xy 92.104751 179.529689) (xy 95.084751 176.549689) (xy 95.094751 111.029689) (xy 98.104751 108.059689)
-        (xy 393.124751 108.049689)
+        (xy 60.184751 200.939689) (xy 60.45 302.51) (xy 50.71 302.66) (xy 46.82 302.66) (xy 47.01 182.74)
+        (xy 46.98 179.06) (xy 92.39 179.05) (xy 94.51 176.57) (xy 94.48 110.95) (xy 94.49 107.31)
+        (xy 396.79 107.28)
       )
     )

Commit message: Added pins for card edge connector
Parts:
- moved J1 1.10 mm to (419.6, 161.3)
Routing:
- net GND: track 9402.9 -> 9439.2 mm
- net COL_B: track 420.3 -> 426.3 mm
- net COL_4: track 550.1 -> 555.9 mm
- net COL_2: track 593.4 -> 599.1 mm
- net COL_F: track 181.6 -> 187.2 mm
- net COL_C: track 414.0 -> 419.6 mm
- net COL_3: track 561.3 -> 566.9 mm
- net COL_5: track 518.8 -> 524.4 mm
- net COL_8: track 512.9 -> 518.4 mm
- net COL_D: track 264.4 -> 269.9 mm
- net COL_9: track 455.6 -> 461.1 mm
- net COL_6: track 525.0 -> 530.4 mm
- net COL_E: track 242.9 -> 248.3 mm
- net COL_A: track 435.6 -> 441.0 mm
- net COL_7: track 487.8 -> 493.1 mm
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
Commit message: Update card edge reader footprint and adjusted / rerouted the connections
Parts:
- moved J1 6.13 mm to (419.0, 167.4)
Connections:
- J1 pad 33: (no net) -> ROW_1
- J1 pad 34: (no net) -> ROW_2
- J1 pad 35: (no net) -> ROW_3
- J1 pad 36: (no net) -> ROW_4
- J1 pad 37: (no net) -> ROW_5
- J1 pad 38: (no net) -> ROW_6
- J1 pad 39: (no net) -> ROW_7
- J1 pad 40: (no net) -> ROW_8
- J1 pad 41: (no net) -> GND
- J1 pad 42: (no net) -> GND
- J1 pad 43: (no net) -> COL_1
- J1 pad 44: (no net) -> COL_2
- J1 pad 45: (no net) -> COL_3
- J1 pad 46: (no net) -> COL_4
- J1 pad 47: (no net) -> COL_5
- J1 pad 48: (no net) -> COL_6
- J1 pad 49: (no net) -> COL_7
- J1 pad 50: (no net) -> COL_8
- J1 pad 51: (no net) -> COL_9
- J1 pad 52: (no net) -> COL_A
- J1 pad 53: (no net) -> COL_B
- J1 pad 54: (no net) -> COL_C
- J1 pad 55: (no net) -> COL_D
- J1 pad 56: (no net) -> COL_E
- J1 pad 57: (no net) -> COL_F
- J1 pad 58: (no net) -> COL_G
- J1 pad 71: (no net) -> GND
- J1 pad 72: (no net) -> GND
Routing:
- net GND: track 9439.2 -> 9474.4 mm
- net COL_G: track 171.8 -> 185.3 mm
- net ROW_6: track 1153.0 -> 1163.3 mm
- net COL_E: track 248.3 -> 256.8 mm
- net COL_9: track 461.1 -> 469.0 mm
- net ROW_1: track 1293.3 -> 1299.4 mm
- net COL_D: track 269.9 -> 275.9 mm
- net ROW_3: track 1260.4 -> 1264.8 mm
- net ROW_5: track 1175.6 -> 1180.0 mm
- net ROW_2: track 1279.3 -> 1283.7 mm
- net ROW_4: track 1249.8 -> 1254.3 mm
- net ROW_8: track 1091.8 -> 1095.3 mm
- net COL_F: track 187.2 -> 190.7 mm
- net ROW_7: track 1093.8 -> 1097.2 mm
- net COL_B: track 426.3 -> 429.4 mm
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Other:
- outline, holes or cut-outs redrawn

Commit message: Added additionnal copper layer on the edges of the PCB
Routing:
- net GND: track 9474.4 -> 9427.4 mm
Other:
- outline, holes or cut-outs redrawn

Commit message: Placed some test points to check continuity of rows and columns
Parts:
- added C1_TEST: TestPoint_Pad_1.0x1.0mm, TestPoint:TestPoint_Pad_1.0x1.0mm, B.Cu at (61.2, 295.4)
- added C2_TEST: TestPoint_Pad_1.0x1.0mm, TestPoint:TestPoint_Pad_1.0x1.0mm, B.Cu at (88.4, 295.4)
- added C3_TEST: TestPoint_Pad_1.0x1.0mm, TestPoint:TestPoint_Pad_1.0x1.0mm, B.Cu at (121.2, 295.4)
- added C4_TEST: TestPoint_Pad_1.0x1.0mm, TestPoint:TestPoint_Pad_1.0x1.0mm, B.Cu at (160.4, 295.4)
- added C5_TEST: TestPoint_Pad_1.0x1.0mm, TestPoint:TestPoint_Pad_1.0x1.0mm, B.Cu at (178.2, 275.1)
- added C6_TEST: TestPoint_Pad_1.0x1.0mm, TestPoint:TestPoint_Pad_1.0x1.0mm, B.Cu at (241.2, 295.5)
- added C7_TEST: TestPoint_Pad_1.0x1.0mm, TestPoint:TestPoint_Pad_1.0x1.0mm, B.Cu at (245.9, 275.1)
- added C8_TEST: TestPoint_Pad_1.0x1.0mm, TestPoint:TestPoint_Pad_1.0x1.0mm, B.Cu at (321.9, 295.6)
- added C9_TEST: TestPoint_Pad_1.0x1.0mm, TestPoint:TestPoint_Pad_1.0x1.0mm, B.Cu at (283.9, 275.1)
- added CA_TEST: TestPoint_Pad_1.0x1.0mm, TestPoint:TestPoint_Pad_1.0x1.0mm, B.Cu at (321.9, 275.1)
- added CB_TEST: TestPoint_Pad_1.0x1.0mm, TestPoint:TestPoint_Pad_1.0x1.0mm, B.Cu at (351.4, 287.4)
- added CC_TEST: TestPoint_Pad_1.0x1.0mm, TestPoint:TestPoint_Pad_1.0x1.0mm, B.Cu at (377.7, 295.4)
- added CD_TEST: TestPoint_Pad_1.0x1.0mm, TestPoint:TestPoint_Pad_1.0x1.0mm, B.Cu at (421.2, 295.5)
- added CE_TEST: TestPoint_Pad_1.0x1.0mm, TestPoint:TestPoint_Pad_1.0x1.0mm, B.Cu at (468.2, 295.6)
- added CF_TEST: TestPoint_Pad_1.0x1.0mm, TestPoint:TestPoint_Pad_1.0x1.0mm, B.Cu at (506.2, 295.5)
- added CG_TEST: TestPoint_Pad_1.0x1.0mm, TestPoint:TestPoint_Pad_1.0x1.0mm, B.Cu at (533.4, 295.6)
- added R1_TEST: TestPoint_Pad_1.0x1.0mm, TestPoint:TestPoint_Pad_1.0x1.0mm, F.Cu at (534.5, 275.5)
- added R2_TEST: TestPoint_Pad_1.0x1.0mm, TestPoint:TestPoint_Pad_1.0x1.0mm, F.Cu at (540.9, 264.8)
- added R3_TEST: TestPoint_Pad_1.0x1.0mm, TestPoint:TestPoint_Pad_1.0x1.0mm, F.Cu at (534.0, 254.5)
- added R4_TEST: TestPoint_Pad_1.0x1.0mm, TestPoint:TestPoint_Pad_1.0x1.0mm, F.Cu at (529.0, 253.4)
- added R5_TEST: TestPoint_Pad_1.0x1.0mm, TestPoint:TestPoint_Pad_1.0x1.0mm, F.Cu at (540.9, 222.8)
- added R6_TEST: TestPoint_Pad_1.0x1.0mm, TestPoint:TestPoint_Pad_1.0x1.0mm, F.Cu at (534.2, 213.0)
- added R7_TEST: TestPoint_Pad_1.0x1.0mm, TestPoint:TestPoint_Pad_1.0x1.0mm, F.Cu at (524.5, 212.0)
- added R8_TEST: TestPoint_Pad_1.0x1.0mm, TestPoint:TestPoint_Pad_1.0x1.0mm, F.Cu at (541.1, 201.8)
Routing:
- net GND: track 9427.4 -> 9490.8 mm
- net COL_E: track 256.8 -> 266.6 mm
- net COL_6: track 533.3 -> 543.1 mm
- net COL_8: track 521.3 -> 531.1 mm
- net COL_D: track 275.9 -> 285.7 mm
- net COL_F: track 190.7 -> 200.4 mm
- net COL_2: track 602.1 -> 611.8 mm
- net COL_C: track 422.5 -> 432.2 mm
- net COL_4: track 559.1 -> 568.7 mm
- net COL_1: track 619.9 -> 629.6 mm
- net COL_3: track 569.8 -> 579.4 mm
- net ROW_7: track 1097.2 -> 1088.2 mm
- net ROW_8: track 1095.3 -> 1102.7 mm
- net ROW_5: track 1180.0 -> 1187.2 mm
- net ROW_2: track 1283.7 -> 1290.9 mm
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